File: edition_one/kicad_5/tiny_modular.sch (KiCad schematic (older format))
At the start: 21 parts, among them J1 Conn_01x01, J2 Conn_01x01, J3 Conn_01x03, J4 Conn_01x06, J5 AudioJack2, J6 AudioJack2, J7 AudioJack2, J8 AudioJack2, SW1 SW_Push, U1 ATtiny85V-10SU

Commit message: Revision anyma 2019 with vertical jack sockets
Parts:
- J5, J6, J7, J8: footprint Custom:AUDIO-JACK-3.5mm_SMD_noHole -> Custom:PJ301M-12_bent; symbol Connector:AudioJack2 -> stahllabs:PJ301M-12
Connections:
- net GND: now also J5.1 (sleeve), J6.1 (sleeve), J7.1 (sleeve), J8.1 (sleeve), RV1.3; no longer J5.S, J6.S, J7.S, J8.S, RV1.1
- net at C1.1, J3.2 (Pin_2), R4.1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: now also RV1.1; no longer RV1.3
- net at J4.2 (Pin_2), R4.2, U1.7 (PB2): now also J7.3 (tip); no longer J7.T
- net at R3.1: now also J8.3 (tip); no longer J8.T
- net at C2.2, R1.1: now also J5.3 (tip), J6.3 (tip); no longer J5.T, J6.T
- no-connect marks 0 -> 4
Changed lines of the file:
@@
 F 3 "~" H 6500 4300 50  0001 C CNN
 	1    6500 4300
-	-1   0    0    1
+	-1   0    0    -1
 $EndComp
 $Comp
@@
 $EndComp
 $Comp
-L Connector:AudioJack2 J5
+L stahllabs:PJ301M-12 J5
 U 1 1 5C804B03
-P 7200 4950
-F 0 "J5" V 7184 5138 50  0000 L CNN
-F 1 "AudioJack2" V 7275 5138 50  0000 L CNN
-F 2 "Custom:AUDIO-JACK-3.5mm_SMD_noHole" H 7200 4950 50  0001 C CNN
-F 3 "~" H 7200 4950 50  0001 C CNN
-	1    7200 4950
+P 7250 5000
+F 0 "J5" V 7234 5188 50  0000 L CNN
+F 1 "AudioJack2" V 7325 5188 50  0000 L CNN
+F 2 "Custom:PJ301M-12_bent" H 7250 5000 50  0001 C CNN
+F 3 "~" H 7250 5000 50  0001 C CNN
+	1    7250 5000
 	0    1    1    0
 $EndComp
@@
 	3500 6200 3500 5850
 $Comp
-L Connector:AudioJack2 J6
+L stahllabs:PJ301M-12 J6
 U 1 1 5C804CF7
-P 8050 4950
-F 0 "J6" V 8034 5138 50  0000 L CNN
-F 1 "AudioJack2" V 8125 5138 50  0000 L CNN
-F 2 "Custom:AUDIO-JACK-3.5mm_SMD_noHole" H 8050 4950 50  0001 C CNN
-F 3 "~" H 8050 4950 50  0001 C CNN
-	1    8050 4950
+P 8100 5000
+F 0 "J6" V 8084 5188 50  0000 L CNN
+F 1 "AudioJack2" V 8175 5188 50  0000 L CNN
+F 2 "Custom:PJ301M-12_bent" H 8100 5000 50  0001 C CNN
+F 3 "~" H 8100 5000 50  0001 C CNN
+	1    8100 5000
 	0    1    1    0
 $EndComp
 $Comp
-L Connector:AudioJack2 J8
+L stahllabs:PJ301M-12 J8
 U 1 1 5C804D2E
-P 9150 4250
-F 0 "J8" V 9134 4438 50  0000 L CNN
-F 1 "AudioJack2" V 9225 4438 50  0000 L CNN
-F 2 "Custom:AUDIO-JACK-3.5mm_SMD_noHole" H 9150 4250 50  0001 C CNN
-F 3 "~" H 9150 4250 50  0001 C CNN
-	1    9150 4250
+P 9150 4300
+F 0 "J8" V 9134 4488 50  0000 L CNN
+F 1 "AudioJack2" V 9225 4488 50  0000 L CNN
+F 2 "Custom:PJ301M-12_bent" H 9150 4300 50  0001 C CNN
+F 3 "~" H 9150 4300 50  0001 C CNN
+	1    9150 4300
 	0    1    1    0
 $EndComp
 $Comp
-L Connector:AudioJack2 J7
+L stahllabs:PJ301M-12 J7
 U 1 1 5C804D65
-P 9150 3400
-F 0 "J7" V 9134 3588 50  0000 L CNN
-F 1 "AudioJack2" V 9225 3588 50  0000 L CNN
-F 2 "Custom:AUDIO-JACK-3.5mm_SMD_noHole" H 9150 3400 50  0001 C CNN
-F 3 "~" H 9150 3400 50  0001 C CNN
-	1    9150 3400
+P 9150 3450
+F 0 "J7" V 9134 3638 50  0000 L CNN
+F 1 "AudioJack2" V 9225 3638 50  0000 L CNN
+F 2 "Custom:PJ301M-12_bent" H 9150 3450 50  0001 C CNN
+F 3 "~" H 9150 3450 50  0001 C CNN
+	1    9150 3450
 	0    1    1    0
 $EndComp
@@
 	7200 2500 7450 2500
 Connection ~ 7200 3750
-Wire Wire Line
-	6500 5850 5600 5850
 Connection ~ 3500 5850
 Wire Wire Line
 	3500 5850 3500 4450
-Wire Wire Line
-	6500 4150 6500 2500
 Connection ~ 6500 2500
 Wire Wire Line
@@
 Wire Wire Line
 	5600 3850 4100 3850
-Wire Wire Line
-	6500 4450 6500 5850
 Wire Wire Line
 	5200 4200 5200 3950
@@
 	4750 4050 4750 1250
 Wire Wire Line
-	6500 5850 7300 5850
-Connection ~ 6500 5850
-Wire Wire Line
-	9150 3600 9150 3750
-Wire Wire Line
-	7200 3750 9150 3750
-Wire Wire Line
-	9250 3600 9250 3750
+	7200 3750 9100 3750
 Wire Wire Line
 	9250 3750 10100 3750
@@
 	2050 5850 3500 5850
 Wire Wire Line
-	7200 5150 7200 5250
-Wire Wire Line
 	7200 5250 8050 5250
-Wire Wire Line
-	8050 5250 8050 5150
 Wire Wire Line
 	7200 5250 5200 5250
@@
 Wire Wire Line
 	5200 5250 5200 5350
-Wire Wire Line
-	7300 5150 7300 5850
-Connection ~ 7300 5850
-Wire Wire Line
-	7300 5850 8150 5850
-Wire Wire Line
-	8150 5150 8150 5850
-Connection ~ 8150 5850
-Wire Wire Line
-	8150 5850 10100 5850
+Connection ~ 7350 5850
+Wire Wire Line
+	7350 5850 8200 5850
+Connection ~ 8200 5850
+Wire Wire Line
+	8200 5850 10100 5850
 Wire Wire Line
 	10100 3750 10100 4700
@@
 	5600 4700 5600 5350
 Wire Wire Line
-	6100 4700 9150 4700
-Wire Wire Line
-	9150 4700 9150 4450
-Wire Wire Line
-	9250 4450 9250 4700
+	6100 4700 9100 4700
 Wire Wire Line
 	9250 4700 10100 4700
@@
 Wire Wire Line
 	2050 1500 2050 2500
-Text Notes 7950 4650 0    50   ~ 0
+Text Notes 7950 4500 0    50   ~ 0
 OUT 2
-Text Notes 7100 4650 0    50   ~ 0
+Text Notes 7100 4500 0    50   ~ 0
 OUT 1
+Wire Wire Line
+	9250 3450 9250 3750
+Wire Wire Line
+	9250 4300 9250 4700
+Wire Wire Line
+	8200 5000 8200 5850
+Wire Wire Line
+	7350 5000 7350 5850
+Wire Wire Line
+	7200 5000 7200 5250
+Wire Wire Line
+	8050 5000 8050 5250
+Wire Wire Line
+	9100 4300 9100 4700
+Wire Wire Line
+	9100 3450 9100 3750
+NoConn ~ 9150 3450
+NoConn ~ 9150 4300
+NoConn ~ 8100 5000
+NoConn ~ 7250 5000
+Wire Wire Line
+	5600 5850 6500 5850
+Wire Wire Line
+	6500 2500 6500 4150
+Wire Wire Line
+	6500 4450 6500 5850
+Connection ~ 6500 5850
+Wire Wire Line
+	6500 5850 7350 5850
 $EndSCHEMATC
